Commit message: added H2O

File: src/usv_sim/urdf/usv.urdf.xacro (robot description, xacro)
@@ -6,4 +6,8 @@
   <xacro:property name="hull_height" value="0.20"/>
   <xacro:property name="camera_size" value="0.08"/>
+  <!-- Water plane size -->
+  <xacro:property name="water_length" value="60.0"/>
+  <xacro:property name="water_width" value="60.0"/>
+  <xacro:property name="water_thickness" value="0.02"/>
   <!-- Base hull -->
   <link name="base_link">
@@ -52,3 +56,20 @@
     <origin xyz="0.30 0.0 0.14" rpy="0 0 0"/>
   </joint>
+  <!-- Water plane -->
+  <link name="water_plane">
+    <visual>
+      <origin xyz="0 0 0" rpy="0 0 0"/>
+      <geometry>
+        <box size="${water_length} ${water_width} ${water_thickness}"/>
+      </geometry>
+      <material name="water_blue">
+        <color rgba="0.0 0.35 0.65 0.55"/>
+      </material>
+    </visual>
+  </link>
+  <joint name="water_joint" type="fixed">
+    <parent link="base_link"/>
+    <child link="water_plane"/>
+    <origin xyz="0 0 -0.12" rpy="0 0 0"/>
+  </joint>
 </robot>

Commit message: final updates to rviz sim and uploaded STL file

File: src/usv_sim/urdf/usv.urdf.xacro (robot description, xacro)
@@ -13,10 +13,10 @@
   <link name="base_link">
     <visual>
-      <origin xyz="0 0 0.0" rpy="0 0 0"/>
+      <origin xyz="-0.5 0.65 -0.25" rpy="1.5708 0 0.0"/>
       <geometry>
-        <box size="${hull_length} ${hull_width} ${hull_height}"/>
+        <mesh filename="package://usv_sim/meshes/boat_hull.STL" scale="1.25 1.25 1.25"/>
       </geometry>
-      <material name="blue">
-        <color rgba="0.1 0.3 0.8 1.0"/>
+      <material name="gray">
+        <color rgba="0.6 0.6 0.6 1.0"/>
       </material>
     </visual>
